File: hardware/BREAD_Slice.kicad_sch (KiCad schematic)
At the start: 16 parts, among them J1 Conn_01x10_Female, J2 Conn_01x08, J3 Conn_01x08

Commit message: completed schematic and board
Parts:
- removed J2, J3: Conn_01x08, TerminalBlock_4Ucon:TerminalBlock_4Ucon_1x08_P3.50mm_Horizontal, symbol Connector_Generic:Conn_01x08
- added J2: Conn_01x03_Pin, Connector_PinHeader_2.54mm:PinHeader_1x03_P2.54mm_Vertical, symbol Connector:Conn_01x03_Pin
- added NT1: NetTie_2, NetTie:NetTie-2_SMD_Pad2.0mm, symbol Device:NetTie_2
- added R1, R2: 1k, Resistor_SMD:R_0603_1608Metric_Pad0.98x0.95mm_HandSolder, symbol Device:R
- D1: PROD_ID (none) -> DIO-12503
- HS1: footprint KML-Custom:Thermal Pad -> kml-custom:Thermal Pad
- U1: value ~ -> AP63205
Connections:
- net D9 is gone; now on net RESET: A1.12 (D9)
- net GND: now also NT1.1; no longer J1.1 (Pin_1), J1.10 (Pin_10), J1.5 (Pin_5)
- net INT: no longer J1.7 (Pin_7)
- net RESET: no longer A1.28 (~{RESET})
- net A0: no longer names the net of A1.19 (A0)
- net A1: no longer names the net of A1.20 (A1)
- net A2: no longer names the net of A1.21 (A2)
- net A3: no longer names the net of A1.22 (A3)
- net A6: no longer names the net of A1.25 (A6)
- net A7: no longer names the net of A1.26 (A7)
- net AREF: no longer names the net of A1.18 (AREF)
- net D10 renamed SS
- net D11 renamed MOSI
- net D12 renamed MISO
- net D13 renamed SCK
- net D6: no longer names the net of A1.9 (D6)
- net D7: no longer names the net of A1.10 (D7)
- net D8: no longer names the net of A1.11 (D8)
- net E_STOP renamed ESTOP
- new net: J2.3 (Pin_3), R2.1
- new net: J2.2 (Pin_2), R1.1
- new net CH19: R1.2
- new net CH20: R2.2
- new net GNDA: J2.1 (Pin_1)
- new net GNDPWR: J1.1 (Pin_1), J1.10 (Pin_10), J1.5 (Pin_5), NT1.2
- no-connect marks 6 -> 19
Other:
- added sheet Dual Selectable SE-DE Thermocouple CJC Input1 (dual_select_thermocouple_input.kicad_sch)
- added sheet Dual Selectable SE-DE Thermocouple CJC Input2 (dual_select_thermocouple_input.kicad_sch)
- added sheet Dual Selectable SE-DE Thermocouple CJC Input3 (dual_select_thermocouple_input.kicad_sch)
- added sheet Dual Selectable SE-DE Thermocouple CJC Input4 (dual_select_thermocouple_input.kicad_sch)
- added sheet Dual Selectable SE-DE Thermocouple CJC Input5 (dual_select_thermocouple_input.kicad_sch)
- added sheet Dual Selectable SE-DE Thermocouple CJC Input6 (dual_select_thermocouple_input.kicad_sch)
- added sheet LTC 2983 Precision Multi-Sensor Temp (ltc2983.kicad_sch)
- added sheet TPS7A4901-5VA (tps7a4901.kicad_sch)
- note added: "5V Switching Supply"
- note added: "Analog 5V"
- note added: "Arduino Nano"
- note added: "Backplane Conn."
- note added: "Clean 5V for analog frontend"
- note added: "Color Scheme Legend: ---------------------------------------------------------- color - value - reference ---------------------------------------------------------- • Red - red3 - Analog 5V Supply (e.g., for amps, ADC, references) • Brown - orange1 - Analog Ground (sensor/amp/ADC ground) • Orange - orange3 - Digital 5V Supply (MCU, digital circuits) • Black - black - Digital Ground (MCU ground) •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"
- note added: "LTC2983 Multi-Sensor Temp System IC"
- note added: "Mounting Holes"
- note added: "Pinout Details Arduino Nano: -------------------------------------------------------------------------------------------------------------------- Pin | Function | Limitations/Notes -------------------------------------------------------------------------------------------------------------------- VIN | External Supply Input | External power source 7-12V GND | Ground | First GND pin available for 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"
- note added: "RGB LED"
- note added: "Thermocouple Inputs Mode Selection Filtering & Protection"
- note added: "removed int from backplane to use with IC int"
- moved on the sheet: A1, C1, C2, C3, C4, H1, H2, H3, H4, L1, U1
