File: hardware/dual_select_thermocouple_input.kicad_sch (KiCad schematic)
At the start: 15 parts, among them J3 PCC-SMP-V-K, J9 PCC-SMP-V-K, Q1 2N3904, SW1 SW_DIP_x03

Commit message: update dip switches to reflect chosen part
Parts:
- SW1: footprint Button_Switch_SMD:SW_DIP_SPSTx03_Slide_6.7x9.18mm_W6.73mm_P2.54mm_LowProfile_JPin -> Button_Switch_SMD:SW_DIP_SPSTx03_Slide_9.78x9.8mm_W8.61mm_P2.54mm
Changed lines of the file:
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@@
 			)
 		)
-		(property "Footprint" "Button_Switch_SMD:SW_DIP_SPSTx03_Slide_6.7x9.18mm_W6.73mm_P2.54mm_LowProfile_JPin"
+		(property "Footprint" "Button_Switch_SMD:SW_DIP_SPSTx03_Slide_9.78x9.8mm_W8.61mm_P2.54mm"
 			(at 86.36 71.12 0)
 			(effects
