File: hardware/dual_select_thermocouple_input.kicad_sch (KiCad schematic)
At the start: 15 parts, among them J3 PCC-SMP-V-K, J9 PCC-SMP-V-K, Q1 2N3904, SW1 SW_DIP_x03

Commit message: chore(hw): migrate KiCad files to the KiCad 10 format
Via `kicad-cli sch upgrade` / `pcb upgrade` (bread-infra
scripts/upgrade_kicad10.sh). Verified lossless: identical netlist, footprint
positions and routing.

Note `sch upgrade` does not cascade into hierarchical sub-sheets, so every
.kicad_sch is upgraded individually -- upgrading only the root sheet leaves
sub-sheets on the old format, which looks migrated and is not.
Parts:
- renumbered C5 to C27, C6 to C28, C7 to C29, D2 to D18, D3 to D19, D4 to D20, D5 to D21, J9 to J13, J3 to J7, Q1 to Q5, R3 to R21, R4 to R22, R5 to R23, R6 to R24, SW1 to SW5

Commit message: fix(hw): re-point stale library nicknames
These parts exist in KiCad-Master-Lib; the boards referenced libraries that no
longer exist (kml-custom, KML-Custom, and SparkFun libraries that never
contained the part) or names the library has since changed.

KiCad embeds footprint geometry in the .kicad_pcb, so the boards rendered and
fabricated correctly and the rot stayed invisible -- it only surfaces on
update-from-library, or when a generator tries to resolve a nickname.

Nickname/name only. No geometry is changed:

  SparkFun-DiscreteSemi:AP63205 -> KMLib_IC_Power:AP63205WU-7_Buck_Regulator
  SparkFun-LED:WS2812-5050-4PIN -> KMLib_IC_SMD:WS2812-5050-4PIN
  kml-custom:DGN8_1P89X1P57 -> KMLib_IC_SMD:DGN8_1P89X1P57
  kml-custom:OMEGA_PCC-SMP-V-K -> KMLib_Connectors:OMEGA_PCC-SMP-V-K
  kml-custom:TPS7A4901DGNR -> KMLib_IC_Power:TPS7A4901DGNR_LDO_Regulator
  kml-custom:Thermal Pad -> KMLib_Mounting:Thermal_Pad

Only references that failed to resolve were touched. Generic parts (<=4 pins)
and KiCad *-rescue libraries are deliberately excluded: fingerprint matching
cannot distinguish a 2-pin resistor from a 2-pin capacitor, so those are being
done by hand.
Parts:
- J13, J7: footprint kml-custom:OMEGA_PCC-SMP-V-K -> KMLib_Connectors:OMEGA_PCC-SMP-V-K
Changed lines of the file:
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@@
 			)
 		)
-		(property "Footprint" "kml-custom:OMEGA_PCC-SMP-V-K"
+		(property "Footprint" "KMLib_Connectors:OMEGA_PCC-SMP-V-K"
 			(at 44.196 48.26 0)
 			(hide yes)
@@
 			)
 		)
-		(property "Footprint" "kml-custom:OMEGA_PCC-SMP-V-K"
+		(property "Footprint" "KMLib_Connectors:OMEGA_PCC-SMP-V-K"
 			(at 44.196 95.25 0)
 			(hide yes)
