File: hardware/BREAD_Slice.kicad_pcb (KiCad board)
At the start: 4 copper layers, 100.1 x 144.9 mm, 124 parts, among them J1 Conn_01x10_Female, J10 PCC-SMP-V-K, J11 PCC-SMP-V-K, J12 PCC-SMP-V-K, J13 PCC-SMP-V-K, J14 PCC-SMP-V-K, J2 Conn_01x03_Pin, J3 PCC-SMP-V-K, J4 PCC-SMP-V-K, J5 PCC-SMP-V-K, J6 PCC-SMP-V-K, J7 PCC-SMP-V-K, J8 PCC-SMP-V-K, J9 PCC-SMP-V-K, Q1 2N3904, Q2 2N3904, Q3 2N3904, Q4 2N3904, Q5 2N3904, Q6 2N3904, SW1 SW_DIP_x03, SW2 SW_DIP_x03, SW3 SW_DIP_x03, SW4 SW_DIP_x03, SW5 SW_DIP_x03, SW6 SW_DIP_x03, U1 AP63205, U2 LTC2983, U3 TPS7A4901DGNR

Commit message: fix(hw): re-point stale library nicknames
These parts exist in KiCad-Master-Lib; the boards referenced libraries that no
longer exist (kml-custom, KML-Custom, and SparkFun libraries that never
contained the part) or names the library has since changed.

KiCad embeds footprint geometry in the .kicad_pcb, so the boards rendered and
fabricated correctly and the rot stayed invisible -- it only surfaces on
update-from-library, or when a generator tries to resolve a nickname.

Nickname/name only. No geometry is changed:

  SparkFun-DiscreteSemi:AP63205 -> KMLib_IC_Power:AP63205WU-7_Buck_Regulator
  SparkFun-LED:WS2812-5050-4PIN -> KMLib_IC_SMD:WS2812-5050-4PIN
  kml-custom:DGN8_1P89X1P57 -> KMLib_IC_SMD:DGN8_1P89X1P57
  kml-custom:OMEGA_PCC-SMP-V-K -> KMLib_Connectors:OMEGA_PCC-SMP-V-K
  kml-custom:TPS7A4901DGNR -> KMLib_IC_Power:TPS7A4901DGNR_LDO_Regulator
  kml-custom:Thermal Pad -> KMLib_Mounting:Thermal_Pad

Only references that failed to resolve were touched. Generic parts (<=4 pins)
and KiCad *-rescue libraries are deliberately excluded: fingerprint matching
cannot distinguish a 2-pin resistor from a 2-pin capacitor, so those are being
done by hand.
Parts:
- D1: footprint SparkFun-LED:WS2812-5050-4PIN -> KMLib_IC_SMD:WS2812-5050-4PIN
- HS1: footprint kml-custom:Thermal Pad -> KMLib_Mounting:Thermal_Pad
- J10, J11, J12, J13, J14, J3, J4, J5, J6, J7, J8, J9: footprint kml-custom:OMEGA_PCC-SMP-V-K -> KMLib_Connectors:OMEGA_PCC-SMP-V-K
- U3: footprint kml-custom:DGN8_1P89X1P57 -> KMLib_IC_SMD:DGN8_1P89X1P57
Changed lines of the file:
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@@
 		)
 	)
-	(footprint "kml-custom:OMEGA_PCC-SMP-V-K"
+	(footprint "KMLib_Connectors:OMEGA_PCC-SMP-V-K"
 		(layer "F.Cu")
 		(at 132.44 101.915 180)
@@
 		)
 	)
-	(footprint "kml-custom:OMEGA_PCC-SMP-V-K"
+	(footprint "KMLib_Connectors:OMEGA_PCC-SMP-V-K"
 		(layer "F.Cu")
 		(at 110.145 61.37 -90)
@@
 		)
 	)
-	(footprint "kml-custom:DGN8_1P89X1P57"
+	(footprint "KMLib_IC_SMD:DGN8_1P89X1P57"
 		(layer "F.Cu")
 		(at 74.509465 121.828932 180)
@@
 		(embedded_fonts no)
 	)
-	(footprint "kml-custom:OMEGA_PCC-SMP-V-K"
+	(footprint "KMLib_Connectors:OMEGA_PCC-SMP-V-K"
 		(layer "F.Cu")
 		(at 132.410001 77.585 180)
@@
 		)
 	)
-	(footprint "SparkFun-LED:WS2812-5050-4PIN"
+	(footprint "KMLib_IC_SMD:WS2812-5050-4PIN"
 		(locked yes)
 		(layer "F.Cu")
@@
 		)
 	)
-	(footprint "kml-custom:OMEGA_PCC-SMP-V-K"
+	(footprint "KMLib_Connectors:OMEGA_PCC-SMP-V-K"
 		(layer "F.Cu")
 		(at 132.34 125.965 180)
@@
 		)
 	)
-	(footprint "kml-custom:OMEGA_PCC-SMP-V-K"
+	(footprint "KMLib_Connectors:OMEGA_PCC-SMP-V-K"
 		(layer "F.Cu")
 		(at 94.475 61.289999 -90)
@@
 		)
 	)
-	(footprint "kml-custom:OMEGA_PCC-SMP-V-K"
+	(footprint "KMLib_Connectors:OMEGA_PCC-SMP-V-K"
 		(layer "F.Cu")
 		(at 132.41 114.36 180)
@@
 		)
 	)
-	(footprint "kml-custom:OMEGA_PCC-SMP-V-K"
+	(footprint "KMLib_Connectors:OMEGA_PCC-SMP-V-K"
 		(layer "F.Cu")
 		(at 122.59 61.4 -90)
@@
 		)
 	)
-	(footprint "kml-custom:Thermal Pad"
+	(footprint "KMLib_Mounting:Thermal_Pad"
 		(layer "F.Cu")
 		(at 66.774465 162.653932)
@@
 		)
 	)
-	(footprint "kml-custom:OMEGA_PCC-SMP-V-K"
+	(footprint "KMLib_Connectors:OMEGA_PCC-SMP-V-K"
 		(layer "F.Cu")
 		(at 132.34 150.295 180)
@@
 		)
 	)
-	(footprint "kml-custom:OMEGA_PCC-SMP-V-K"
+	(footprint "KMLib_Connectors:OMEGA_PCC-SMP-V-K"
 		(layer "F.Cu")
 		(at 132.31 138.41 180)
@@
 		(embedded_fonts no)
 	)
-	(footprint "kml-custom:OMEGA_PCC-SMP-V-K"
+	(footprint "KMLib_Connectors:OMEGA_PCC-SMP-V-K"
 		(layer "F.Cu")
 		(at 132.31 162.74 180)
@@
 		)
 	)
-	(footprint "kml-custom:OMEGA_PCC-SMP-V-K"
+	(footprint "KMLib_Connectors:OMEGA_PCC-SMP-V-K"
 		(layer "F.Cu")
 		(at 82.03 61.259998 -90)
@@
 		)
 	)
-	(footprint "kml-custom:OMEGA_PCC-SMP-V-K"
+	(footprint "KMLib_Connectors:OMEGA_PCC-SMP-V-K"
 		(layer "F.Cu")
 		(at 132.38 90.03 180)
