File: hardware/tps7a4901.kicad_sch (KiCad schematic)
At the start: 8 parts, among them U3 TPS7A4901DGNR

Commit message: fix(hw): re-point stale library nicknames
These parts exist in KiCad-Master-Lib; the boards referenced libraries that no
longer exist (kml-custom, KML-Custom, and SparkFun libraries that never
contained the part) or names the library has since changed.

KiCad embeds footprint geometry in the .kicad_pcb, so the boards rendered and
fabricated correctly and the rot stayed invisible -- it only surfaces on
update-from-library, or when a generator tries to resolve a nickname.

Nickname/name only. No geometry is changed:

  SparkFun-DiscreteSemi:AP63205 -> KMLib_IC_Power:AP63205WU-7_Buck_Regulator
  SparkFun-LED:WS2812-5050-4PIN -> KMLib_IC_SMD:WS2812-5050-4PIN
  kml-custom:DGN8_1P89X1P57 -> KMLib_IC_SMD:DGN8_1P89X1P57
  kml-custom:OMEGA_PCC-SMP-V-K -> KMLib_Connectors:OMEGA_PCC-SMP-V-K
  kml-custom:TPS7A4901DGNR -> KMLib_IC_Power:TPS7A4901DGNR_LDO_Regulator
  kml-custom:Thermal Pad -> KMLib_Mounting:Thermal_Pad

Only references that failed to resolve were touched. Generic parts (<=4 pins)
and KiCad *-rescue libraries are deliberately excluded: fingerprint matching
cannot distinguish a 2-pin resistor from a 2-pin capacitor, so those are being
done by hand.
Parts:
- U3: footprint kml-custom:DGN8_1P89X1P57 -> KMLib_IC_SMD:DGN8_1P89X1P57; symbol kml-custom:TPS7A4901DGNR -> KMLib_IC_Power:TPS7A4901DGNR_LDO_Regulator
Changed lines of the file:
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@@
 	)
 	(symbol
-		(lib_id "kml-custom:TPS7A4901DGNR")
+		(lib_id "KMLib_IC_Power:TPS7A4901DGNR_LDO_Regulator")
 		(at 180.34 90.17 0)
 		(mirror y)
@@
 			)
 		)
-		(property "Footprint" "kml-custom:DGN8_1P89X1P57"
+		(property "Footprint" "KMLib_IC_SMD:DGN8_1P89X1P57"
 			(at 160.02 90.17 0)
 			(hide yes)
